File: Envoy/Envoy.sch (KiCad schematic (older format))
At the start: 53 parts, among them U1 ProMicro

Commit message: Rev 0.2 including switchplate and backplate
Parts:
- added H1, H2, H3, H4: MountingHole, Envoy:ClearanceHole_3.7mm, symbol Mechanical:MountingHole
- ENC1, ENC2: footprint Keebio_parts:RotaryEncoder_EC11 -> Keebio-Parts:RotaryEncoder_EC11-no-legs
- MX1, MX10, MX11, MX13, MX14, MX15, MX19, MX2, MX3, MX4, MX5, MX6, MX7, MX9: footprint MX_Only:MXOnly-1U-Hotswap -> Envoy:MXOnly-1U-Hotswap
- MX18: footprint Envoy:MXOnly-1U-Hotswap-2KeyAlternativeLeft -> Envoy:MXOnly-1U-HotswapReversed-2KeyAlternativeLeft
Connections:
- net GND: now also RESET1.1; no longer RESET1.2
- net col1: now also U1.18 (F6/A1); no longer U1.17 (F7/A0)
- net col2: now also U1.17 (F7/A0); no longer U1.13 (B6/10)
- net col3: now also U1.16 (B1/15); no longer U1.15 (B3/14)
- net col4: now also U1.11 (8/B4); no longer U1.12 (9/B5)
- net enc1A: now also U1.1 (TX0/D3); no longer U1.2 (RX1/D2)
- net enc1B: now also U1.2 (RX1/D2); no longer U1.1 (TX0/D3)
- net reset: now also RESET1.2; no longer RESET1.1
- net row1: now also U1.13 (B6/10); no longer U1.18 (F6/A1)
- net row3: now also U1.15 (B3/14); no longer U1.16 (B1/15)
- net row4: now also U1.12 (9/B5); no longer U1.11 (8/B4)
Changed lines of the file:
@@
 F 0 "MX1" H 4783 2823 60  0000 C CNN
 F 1 "MX-NoLED" H 4783 2749 20  0000 C CNN
-F 2 "MX_Only:MXOnly-1U-Hotswap" H 4125 2575 60  0001 C CNN
+F 2 "Envoy:MXOnly-1U-Hotswap" H 4125 2575 60  0001 C CNN
 F 3 "" H 4125 2575 60  0001 C CNN
 	1    4750 2600
@@
 F 0 "MX2" H 5433 2823 60  0000 C CNN
 F 1 "MX-NoLED" H 5433 2749 20  0000 C CNN
-F 2 "MX_Only:MXOnly-1U-Hotswap" H 4775 2575 60  0001 C CNN
+F 2 "Envoy:MXOnly-1U-Hotswap" H 4775 2575 60  0001 C CNN
 F 3 "" H 4775 2575 60  0001 C CNN
 	1    5400 2600
@@
 F 0 "MX3" H 6083 2823 60  0000 C CNN
 F 1 "MX-NoLED" H 6083 2749 20  0000 C CNN
-F 2 "MX_Only:MXOnly-1U-Hotswap" H 5425 2575 60  0001 C CNN
+F 2 "Envoy:MXOnly-1U-Hotswap" H 5425 2575 60  0001 C CNN
 F 3 "" H 5425 2575 60  0001 C CNN
 	1    6050 2600
@@
 F 0 "MX4" H 6683 2823 60  0000 C CNN
 F 1 "MX-NoLED" H 6683 2749 20  0000 C CNN
-F 2 "MX_Only:MXOnly-1U-Hotswap" H 6025 2575 60  0001 C CNN
+F 2 "Envoy:MXOnly-1U-Hotswap" H 6025 2575 60  0001 C CNN
 F 3 "" H 6025 2575 60  0001 C CNN
 	1    6650 2600
@@
 F 0 "MX11" H 6083 3823 60  0000 C CNN
 F 1 "MX-NoLED" H 6083 3749 20  0000 C CNN
-F 2 "MX_Only:MXOnly-1U-Hotswap" H 5425 3575 60  0001 C CNN
+F 2 "Envoy:MXOnly-1U-Hotswap" H 5425 3575 60  0001 C CNN
 F 3 "" H 5425 3575 60  0001 C CNN
 	1    6050 3600
@@
 F 0 "MX10" H 5433 3823 60  0000 C CNN
 F 1 "MX-NoLED" H 5433 3749 20  0000 C CNN
-F 2 "MX_Only:MXOnly-1U-Hotswap" H 4775 3575 60  0001 C CNN
+F 2 "Envoy:MXOnly-1U-Hotswap" H 4775 3575 60  0001 C CNN
 F 3 "" H 4775 3575 60  0001 C CNN
 	1    5400 3600
@@
 F 0 "MX9" H 4783 3823 60  0000 C CNN
 F 1 "MX-NoLED" H 4783 3749 20  0000 C CNN
-F 2 "MX_Only:MXOnly-1U-Hotswap" H 4125 3575 60  0001 C CNN
+F 2 "Envoy:MXOnly-1U-Hotswap" H 4125 3575 60  0001 C CNN
 F 3 "" H 4125 3575 60  0001 C CNN
 	1    4750 3600
@@
 F 0 "MX7" H 6083 3323 60  0000 C CNN
 F 1 "MX-NoLED" H 6083 3249 20  0000 C CNN
-F 2 "MX_Only:MXOnly-1U-Hotswap" H 5425 3075 60  0001 C CNN
+F 2 "Envoy:MXOnly-1U-Hotswap" H 5425 3075 60  0001 C CNN
 F 3 "" H 5425 3075 60  0001 C CNN
 	1    6050 3100
@@
 F 0 "MX6" H 5433 3323 60  0000 C CNN
 F 1 "MX-NoLED" H 5433 3249 20  0000 C CNN
-F 2 "MX_Only:MXOnly-1U-Hotswap" H 4775 3075 60  0001 C CNN
+F 2 "Envoy:MXOnly-1U-Hotswap" H 4775 3075 60  0001 C CNN
 F 3 "" H 4775 3075 60  0001 C CNN
 	1    5400 3100
@@
 F 0 "MX5" H 4783 3323 60  0000 C CNN
 F 1 "MX-NoLED" H 4783 3249 20  0000 C CNN
-F 2 "MX_Only:MXOnly-1U-Hotswap" H 4125 3075 60  0001 C CNN
+F 2 "Envoy:MXOnly-1U-Hotswap" H 4125 3075 60  0001 C CNN
 F 3 "" H 4125 3075 60  0001 C CNN
 	1    4750 3100
@@
 F 0 "MX15" H 6083 4323 60  0000 C CNN
 F 1 "MX-NoLED" H 6083 4249 20  0000 C CNN
-F 2 "MX_Only:MXOnly-1U-Hotswap" H 5425 4075 60  0001 C CNN
+F 2 "Envoy:MXOnly-1U-Hotswap" H 5425 4075 60  0001 C CNN
 F 3 "" H 5425 4075 60  0001 C CNN
 	1    6050 4100
@@
 F 0 "MX14" H 5433 4323 60  0000 C CNN
 F 1 "MX-NoLED" H 5433 4249 20  0000 C CNN
-F 2 "MX_Only:MXOnly-1U-Hotswap" H 4775 4075 60  0001 C CNN
+F 2 "Envoy:MXOnly-1U-Hotswap" H 4775 4075 60  0001 C CNN
 F 3 "" H 4775 4075 60  0001 C CNN
 	1    5400 4100
@@
 F 0 "MX13" H 4783 4323 60  0000 C CNN
 F 1 "MX-NoLED" H 4783 4249 20  0000 C CNN
-F 2 "MX_Only:MXOnly-1U-Hotswap" H 4125 4075 60  0001 C CNN
+F 2 "Envoy:MXOnly-1U-Hotswap" H 4125 4075 60  0001 C CNN
 F 3 "" H 4125 4075 60  0001 C CNN
 	1    4750 4100
@@
 F 0 "MX19" H 6083 4823 60  0000 C CNN
 F 1 "MX-NoLED" H 6083 4749 20  0000 C CNN
-F 2 "MX_Only:MXOnly-1U-Hotswap" H 5425 4575 60  0001 C CNN
+F 2 "Envoy:MXOnly-1U-Hotswap" H 5425 4575 60  0001 C CNN
 F 3 "" H 5425 4575 60  0001 C CNN
 	1    6050 4600
@@
 F 0 "MX18" H 5433 4823 60  0000 C CNN
 F 1 "MX-NoLED" H 5433 4749 20  0000 C CNN
-F 2 "Envoy:MXOnly-1U-Hotswap-2KeyAlternativeLeft" H 4775 4575 60  0001 C CNN
+F 2 "Envoy:MXOnly-1U-HotswapReversed-2KeyAlternativeLeft" H 4775 4575 60  0001 C CNN
 F 3 "" H 4775 4575 60  0001 C CNN
 	1    5400 4600
@@
 Text GLabel 4350 3300 0    50   Input ~ 0
 row1
-Text GLabel 2850 2200 2    50   Input ~ 0
+Text GLabel 2850 2700 2    50   Input ~ 0
 row1
 Text GLabel 2850 2600 2    50   Input ~ 0
 row2
-Text GLabel 2850 2400 2    50   Input ~ 0
+Text GLabel 2850 2500 2    50   Input ~ 0
 row3
-Text GLabel 1450 2600 0    50   Input ~ 0
+Text GLabel 1450 2700 0    50   Input ~ 0
 row4
 Text GLabel 2850 2100 2    50   Input ~ 0
 col0
+Text GLabel 2850 2200 2    50   Input ~ 0
+col1
 Text GLabel 2850 2300 2    50   Input ~ 0
-col1
-Text GLabel 2850 2700 2    50   Input ~ 0
 col2
-Text GLabel 2850 2500 2    50   Input ~ 0
+Text GLabel 2850 2400 2    50   Input ~ 0
 col3
 Text GLabel 2850 1800 2    50   Input ~ 0
@@
 F 0 "ENC1" V 7854 2880 50  0000 L CNN
 F 1 "Rotary_Encoder_Switch" V 7945 2880 50  0000 L CNN
-F 2 "Keebio_parts:RotaryEncoder_EC11" H 7750 2810 50  0001 C CNN
+F 2 "Keebio-Parts:RotaryEncoder_EC11-no-legs" H 7750 2810 50  0001 C CNN
 F 3 "~" H 7900 2910 50  0001 C CNN
 	1    7900 2650
@@
 F 0 "ENC2" V 7854 3380 50  0000 L CNN
 F 1 "Rotary_Encoder_Switch" V 7945 3380 50  0000 L CNN
-F 2 "Keebio_parts:RotaryEncoder_EC11" H 7750 3310 50  0001 C CNN
+F 2 "Keebio-Parts:RotaryEncoder_EC11-no-legs" H 7750 3310 50  0001 C CNN
 F 3 "~" H 7900 3410 50  0001 C CNN
 	1    7900 3150
@@
 	4500 4800 5150 4800
 Connection ~ 5150 4800
-Text GLabel 1450 2700 0    50   Input ~ 0
+Text GLabel 1450 2600 0    50   Input ~ 0
 col4
 Text GLabel 8200 2750 2    50   Input ~ 0
@@
 Text GLabel 8200 4050 2    50   Input ~ 0
 enc4B
+Text GLabel 1450 1600 0    50   Input ~ 0
+enc1A
 Text GLabel 1450 1700 0    50   Input ~ 0
-enc1A
-Text GLabel 1450 1600 0    50   Input ~ 0
 enc1B
 Text GLabel 1450 2100 0    50   Input ~ 0
@@
 L power:GND #PWR0104
 U 1 1 6162407C
-P 2350 3500
-F 0 "#PWR0104" H 2350 3250 50  0001 C CNN
-F 1 "GND" H 2355 3327 50  0000 C CNN
-F 2 "" H 2350 3500 50  0001 C CNN
-F 3 "" H 2350 3500 50  0001 C CNN
-	1    2350 3500
-	1    0    0    -1
-$EndComp
-Text GLabel 1750 3500 0    50   Input ~ 0
+P 1750 3500
+F 0 "#PWR0104" H 1750 3250 50  0001 C CNN
+F 1 "GND" H 1755 3327 50  0000 C CNN
+F 2 "" H 1750 3500 50  0001 C CNN
+F 3 "" H 1750 3500 50  0001 C CNN
+	1    1750 3500
+	1    0    0    -1
+$EndComp
+Text GLabel 2350 3500 2    50   Input ~ 0
 reset
 $Comp
@@
 Text GLabel 1450 2000 0    50   Input ~ 0
 enc2B
+$Comp
+L Mechanical:MountingHole H1
+U 1 1 618E522A
+P 3850 1150
+F 0 "H1" H 3950 1196 50  0000 L CNN
+F 1 "MountingHole" H 3950 1105 50  0000 L CNN
+F 2 "Envoy:ClearanceHole_3.7mm" H 3850 1150 50  0001 C CNN
+F 3 "~" H 3850 1150 50  0001 C CNN
+	1    3850 1150
+	1    0    0    -1
+$EndComp
+$Comp
+L Mechanical:MountingHole H2
+U 1 1 618E614F
+P 3850 1350
+F 0 "H2" H 3950 1396 50  0000 L CNN
+F 1 "MountingHole" H 3950 1305 50  0000 L CNN
+F 2 "Envoy:ClearanceHole_3.7mm" H 3850 1350 50  0001 C CNN
+F 3 "~" H 3850 1350 50  0001 C CNN
+	1    3850 1350
+	1    0    0    -1
+$EndComp
+$Comp
+L Mechanical:MountingHole H3
+U 1 1 618E7016
+P 3850 1550
+F 0 "H3" H 3950 1596 50  0000 L CNN
+F 1 "MountingHole" H 3950 1505 50  0000 L CNN
+F 2 "Envoy:ClearanceHole_3.7mm" H 3850 1550 50  0001 C CNN
+F 3 "~" H 3850 1550 50  0001 C CNN
+	1    3850 1550
+	1    0    0    -1
+$EndComp
+$Comp
+L Mechanical:MountingHole H4
+U 1 1 618E7362
+P 3850 1750
+F 0 "H4" H 3950 1796 50  0000 L CNN
+F 1 "MountingHole" H 3950 1705 50  0000 L CNN
+F 2 "Envoy:ClearanceHole_3.7mm" H 3850 1750 50  0001 C CNN
+F 3 "~" H 3850 1750 50  0001 C CNN
+	1    3850 1750
+	1    0    0    -1
+$EndComp
 $EndSCHEMATC
