File: Envoy/Envoy.kicad_sch (KiCad schematic)
At the start: 57 parts

Commit message: More tweaks to the switchplate cutouts, make switchplate float instead of the PCB, move diodes to give more space to stabs
Parts:
- H1, H2, H3, H4: footprint Envoy:ClearanceHole_3.7mm -> MountingHole:MountingHole_2.5mm
- MX15: footprint Envoy:MXOnly-1U-HotswapReversed -> Envoy:MXOnly-1U-Hotswap
- MX20: footprint Envoy:MXOnly-1U-Hotswap-2KeyAlternativeLeft -> Envoy:MXOnly-1U-HotswapReversed-2KeyAlternativeLeft
- MX4: footprint Envoy:MXOnly-1U-Hotswap -> Envoy:MXOnly-1U-HotswapReversed
Changed lines of the file:
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@@
       (effects (font (size 1.27 1.27)) (justify left))
     )
-    (property "Footprint" "Envoy:ClearanceHole_3.7mm" (id 2) (at 97.79 29.21 0)
+    (property "Footprint" "MountingHole:MountingHole_2.5mm" (id 2) (at 97.79 29.21 0)
       (effects (font (size 1.27 1.27)) hide)
     )
@@
       (effects (font (size 1.27 1.27)) (justify left))
     )
-    (property "Footprint" "Envoy:ClearanceHole_3.7mm" (id 2) (at 97.79 34.29 0)
+    (property "Footprint" "MountingHole:MountingHole_2.5mm" (id 2) (at 97.79 34.29 0)
       (effects (font (size 1.27 1.27)) hide)
     )
@@
       (effects (font (size 1.27 1.27)) (justify left))
     )
-    (property "Footprint" "Envoy:ClearanceHole_3.7mm" (id 2) (at 97.79 39.37 0)
+    (property "Footprint" "MountingHole:MountingHole_2.5mm" (id 2) (at 97.79 39.37 0)
       (effects (font (size 1.27 1.27)) hide)
     )
@@
       (effects (font (size 1.27 1.27)) (justify left))
     )
-    (property "Footprint" "Envoy:ClearanceHole_3.7mm" (id 2) (at 97.79 44.45 0)
+    (property "Footprint" "MountingHole:MountingHole_2.5mm" (id 2) (at 97.79 44.45 0)
       (effects (font (size 1.27 1.27)) hide)
     )
@@
       (effects (font (size 0.508 0.508)))
     )
-    (property "Footprint" "Envoy:MXOnly-1U-HotswapReversed" (id 2) (at 137.795 104.775 0)
+    (property "Footprint" "Envoy:MXOnly-1U-Hotswap" (id 2) (at 137.795 104.775 0)
       (effects (font (size 1.524 1.524)) hide)
     )
@@
       (effects (font (size 0.508 0.508)))
     )
-    (property "Footprint" "Envoy:MXOnly-1U-Hotswap" (id 2) (at 153.035 66.675 0)
+    (property "Footprint" "Envoy:MXOnly-1U-HotswapReversed" (id 2) (at 153.035 66.675 0)
       (effects (font (size 1.524 1.524)) hide)
     )
@@
       (effects (font (size 0.508 0.508)))
     )
-    (property "Footprint" "Envoy:MXOnly-1U-Hotswap-2KeyAlternativeLeft" (id 2) (at 153.035 117.475 0)
+    (property "Footprint" "Envoy:MXOnly-1U-HotswapReversed-2KeyAlternativeLeft" (id 2) (at 153.035 117.475 0)
       (effects (font (size 1.524 1.524)) hide)
     )
@@
     )
     (path "/00000000-0000-0000-0000-0000618e522a"
-      (reference "H1") (unit 1) (value "MountingHole") (footprint "Envoy:ClearanceHole_3.7mm")
+      (reference "H1") (unit 1) (value "MountingHole") (footprint "MountingHole:MountingHole_2.5mm")
     )
     (path "/00000000-0000-0000-0000-0000618e614f"
-      (reference "H2") (unit 1) (value "MountingHole") (footprint "Envoy:ClearanceHole_3.7mm")
+      (reference "H2") (unit 1) (value "MountingHole") (footprint "MountingHole:MountingHole_2.5mm")
     )
     (path "/00000000-0000-0000-0000-0000618e7016"
-      (reference "H3") (unit 1) (value "MountingHole") (footprint "Envoy:ClearanceHole_3.7mm")
+      (reference "H3") (unit 1) (value "MountingHole") (footprint "MountingHole:MountingHole_2.5mm")
     )
     (path "/00000000-0000-0000-0000-0000618e7362"
-      (reference "H4") (unit 1) (value "MountingHole") (footprint "Envoy:ClearanceHole_3.7mm")
+      (reference "H4") (unit 1) (value "MountingHole") (footprint "MountingHole:MountingHole_2.5mm")
     )
     (path "/00000000-0000-0000-0000-000061511883"
@@
     )
     (path "/00000000-0000-0000-0000-00006152424a"
-      (reference "MX4") (unit 1) (value "MX-NoLED") (footprint "Envoy:MXOnly-1U-Hotswap")
+      (reference "MX4") (unit 1) (value "MX-NoLED") (footprint "Envoy:MXOnly-1U-HotswapReversed")
     )
     (path "/00000000-0000-0000-0000-00006152049e"
@@
     )
     (path "/00000000-0000-0000-0000-00006152d914"
-      (reference "MX15") (unit 1) (value "MX-NoLED") (footprint "Envoy:MXOnly-1U-HotswapReversed")
+      (reference "MX15") (unit 1) (value "MX-NoLED") (footprint "Envoy:MXOnly-1U-Hotswap")
     )
     (path "/00000000-0000-0000-0000-00006152d8fc"
@@
     )
     (path "/00000000-0000-0000-0000-0000615324b8"
-      (reference "MX20") (unit 1) (value "MX-NoLED") (footprint "Envoy:MXOnly-1U-Hotswap-2KeyAlternativeLeft")
+      (reference "MX20") (unit 1) (value "MX-NoLED") (footprint "Envoy:MXOnly-1U-HotswapReversed-2KeyAlternativeLeft")
     )
     (path "/00000000-0000-0000-0000-00006150d40a"
