File: Envoy/Envoy-Backplate/_autosave-Envoy-Backplate.kicad_pcb (KiCad board)
At the start: 2 copper layers, 95.4 x 95.4 mm, 13 parts

Commit message: Fix switchplate cutout sizes
Parts:
- moved H1 4.75 mm to (123.4, 85.4)
Changed lines of the file:
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@@
   )
   (footprint "Envoy:MountingHole_Reinforced_2.5mm" (layer "F.Cu")
-    (at 128.175 85.37575)
+    (at 123.425 85.37575)
     (descr "Mounting Hole 2.5mm, no annular")
     (tags "mounting hole 2.5mm no annular")
